File: Analog_Computer_Rack_Power_Filter.kicad_sch (KiCad schematic)
At the start: 24 parts, among them J1 Screw_Terminal_01x02, J2 Screw_Terminal_01x02, J3 Screw_Terminal_01x02, J4 Screw_Terminal_01x02, M1 Q_PNP_Darlington_BCE, Q1 Q_NPN_Darlington_BCE, Q2 LM340T-12/NOPB, Q3 LM7912CT

Commit message: finished Version V1
Parts:
- removed C3, C4, C5, C6: 160µ, symbol Device:C
- added C3, C4, C5, C9: C_Polarized, Capacitor_THT:CP_Radial_D12.5mm_P5.00mm, symbol Device:C_Polarized
- added H1, H2, H3, H4: MountingHole, MountingHole:MountingHole_3.2mm_M3_DIN965, symbol Mechanical:MountingHole
- C1, C7: value C -> 2.2u; footprint (none) -> Capacitor_THT:C_Rect_L4.6mm_W3.0mm_P2.50mm_MKS02_FKP02
- C2, C8: value C -> 1u; footprint (none) -> Capacitor_THT:C_Rect_L4.6mm_W3.0mm_P2.50mm_MKS02_FKP02
- J1, J2, J3, J4: footprint (none) -> analog_computing:TerminalBlock_TB003-500-P02BE
- R1, R3, R4: value 100 -> 1k; footprint (none) -> Resistor_THT:R_Axial_DIN0207_L6.3mm_D2.5mm_P7.62mm_Horizontal
- R2: value R -> 1k; footprint (none) -> Resistor_THT:R_Axial_DIN0207_L6.3mm_D2.5mm_P7.62mm_Horizontal
Connections:
- net GND: now also C3.2, C4.1, C5.1, C9.2
- net at M1.1 (B), R4.2: now also C5.2
- net at R3.2, R4.1: now also C4.2
- net at R1.2, R2.1: now also C9.1
- net at Q1.1 (B), R2.2: now also C3.1
Other:
- note added: "Mountingholes"
- note added: "TB003-500-P02BE"
